Commit message: Add zed cam startup scripts and slam

File: rbpodo_description/robots/rb10_1300e.urdf (robot description, URDF)
Before this commit: robot rb10_1300e, 8 links, 7 joints
Links:
- added link camera_mount_link, mass 0.072; collision box size=0.030 0.095 0.030; visual box size=0.025 0.090 0.025
Joints:
- added joint link6_to_camera_mount: type fixed, parent link6, child camera_mount_link, origin xyz=0.0 0.0 0.0 rpy=0.0 0.0 0.0

File: rbpodo_description/robots/rb10_1300e.urdf.xacro (robot description, xacro)
@@ -8,4 +8,20 @@
   <xacro:arg name="use_fake_hardware" default="true"/>
   <xacro:arg name="fake_sensor_commands" default="false"/>
+  <!-- Stereolabs ZED Mini (USB 3, direct-attached) on link6.
+       Default orientation mirrors aw_description/urdf/aw_camera_mount.xacro:
+         zedm +X (lens look) = link6 −Y
+       so the mount uses rpy=(0, 0, −pi/2). -->
+  <!-- Camera mounted on top of TCP, lens facing forward (tcp -Y direction).
+       ZED +X = lens direction → yaw -pi/2 maps cam +X to tcp -Y. -->
+  <xacro:arg name="cam_x" default="0.0"/>
+  <xacro:arg name="cam_y" default="-0.13"/>
+  <xacro:arg name="cam_z" default="0.10"/>
+  <xacro:arg name="cam_roll" default="0.0"/>
+  <!-- 25 degrees up -->
+  <!-- <xacro:arg name="cam_pitch" default="0.436332"/>   -->
+  <!-- 22.5 degrees up -->
+  <xacro:arg name="cam_pitch" default=".3926996332"/>
+  <!-- <xacro:arg name="cam_yaw" default="-1.5707963267948966"/> -->
+  <xacro:arg name="cam_yaw" default="-1.5707963267948966"/>
   <!-- torque_constant = actual_torque_constant * gear_ratio -->
   <xacro:property name="base_tc" value="${1}" />
@@ -17,3 +33,45 @@
   <xacro:rb_6dof model_id="rb10_1300e" prefix="$(arg prefix)" tcp_name="tcp" tcp_xyz="0 -0.1153 0" tcp_rpy="0 0 0" />
   <xacro:rb_6dof_ros2_control prefix="$(arg prefix)" robot_ip="$(arg robot_ip)" cb_simulation="$(arg cb_simulation)" use_fake_hardware="$(arg use_fake_hardware)" fake_sensor_commands="$(arg fake_sensor_commands)" torque_constants="${[base_tc, shoulder_tc, elbow_tc, wrist1_tc, wrist2_tc, wrist3_tc]}" />
+  <!-- ══════════════════════════════════════════════════════════════════
+       ZED Mini mount — SELF-CONTAINED.
+       This file used to include `zed_macro.urdf.xacro`, which in turn tried
+       to load `$(find zed_msgs)/meshes/zedm.stl`. On machines where that mesh
+       package/path is missing, RViz reports:
+         "Error retrieving file ... meshes/zedm.stl"
+       and the camera body disappears.
+       To make the robot description robust everywhere, we inline the same
+       ZED frame chain here and render the body as a simple box sized to the
+       real ZED Mini (124.5 x 30.5 x 26.5 mm). The frame names remain identical
+       to Stereolabs' macro so downstream TF/topic consumers still work.
+       Orientation rule for this rig:
+         zedm +X (lens look) = link6 -Y
+       so the mount uses rpy=(0, 0, -pi/2).
+       ══════════════════════════════════════════════════════════════════ -->
+  <xacro:property name="M_PI" value="3.1415926535897931"/>
+  <link name="$(arg prefix)camera_mount_link">
+    <visual>
+      <origin xyz="0 0 0" rpy="0 0 0"/>
+      <geometry>
+        <mesh filename="package://rbpodo_description/meshes/sensors/zedm.stl"/>
+      </geometry>
+      <material name="dark_grey">
+        <color rgba="0.25 0.25 0.25 1.0"/>
+      </material>
+    </visual>
+    <collision>
+      <geometry>
+        <box size="0.030 0.095 0.030"/>
+      </geometry>
+    </collision>
+    <inertial>
+      <mass value="0.072"/>
+      <inertia ixx="0.00001" ixy="0.0" ixz="0.0" iyy="0.00001" iyz="0.0" izz="0.00001"/>
+    </inertial>
+  </link>
+  <joint name="$(arg prefix)link6_to_camera_mount" type="fixed">
+    <parent link="$(arg prefix)link6"/>
+    <child link="$(arg prefix)camera_mount_link"/>
+    <origin xyz="$(arg cam_x) $(arg cam_y) $(arg cam_z)"
+            rpy="$(arg cam_roll) $(arg cam_pitch) $(arg cam_yaw)"/>
+  </joint>
 </robot>

File: rbpodo_description/robots/rb10_1300e_u.urdf (robot description, URDF)
Before this commit: robot rb10_1300e_u, 8 links, 7 joints
Links:
- added link camera_mount_link, mass 0.072; collision box size=0.030 0.095 0.030; visual box size=0.025 0.090 0.025
Joints:
- added joint link6_to_camera_mount: type fixed, parent link6, child camera_mount_link, origin xyz=0 -0.08 0 rpy=0 0 -1.5707963267948966

File: rbpodo_description/robots/rb10_1300e_u.urdf.xacro (robot description, xacro)
@@ -8,4 +8,12 @@
   <xacro:arg name="use_fake_hardware" default="true"/>
   <xacro:arg name="fake_sensor_commands" default="false"/>
+  <!-- Stereolabs ZED Mini on link6 — same mount as rb10_1300e.urdf.xacro.
+       Lens look (zedm +X) = link6 −Y  →  rpy=(0, 0, −π/2) on link6→camera_mount. -->
+  <xacro:arg name="cam_x" default="0.0"/>
+  <xacro:arg name="cam_y" default="-0.08"/>
+  <xacro:arg name="cam_z" default="0.0"/>
+  <xacro:arg name="cam_roll" default="0.0"/>
+  <xacro:arg name="cam_pitch" default="0.0"/>
+  <xacro:arg name="cam_yaw" default="-1.5707963267948966"/>
   <!-- torque_constant = actual_torque_constant * gear_ratio -->
   <xacro:property name="base_tc" value="${1}" />
@@ -17,3 +25,32 @@
   <xacro:rb_6dof model_id="rb10_1300e_u" prefix="$(arg prefix)" tcp_name="tcp" tcp_xyz="0 -0.1153 0" tcp_rpy="0 0 0" />
   <xacro:rb_6dof_ros2_control prefix="$(arg prefix)" robot_ip="$(arg robot_ip)" cb_simulation="$(arg cb_simulation)" use_fake_hardware="$(arg use_fake_hardware)" fake_sensor_commands="$(arg fake_sensor_commands)" torque_constants="${[base_tc, shoulder_tc, elbow_tc, wrist1_tc, wrist2_tc, wrist3_tc]}" />
+  <!-- ══════════════════════════════════════════════════════════════════
+       ZED Mini mount — SELF-CONTAINED (no zed_msgs STL). Matches rb10_1300e.
+       ══════════════════════════════════════════════════════════════════ -->
+  <xacro:property name="M_PI" value="3.1415926535897931"/>
+  <link name="$(arg prefix)camera_mount_link">
+    <visual>
+      <geometry>
+        <box size="0.025 0.090 0.025"/>
+      </geometry>
+      <material name="dark_grey">
+        <color rgba="0.3 0.3 0.3 1.0"/>
+      </material>
+    </visual>
+    <collision>
+      <geometry>
+        <box size="0.030 0.095 0.030"/>
+      </geometry>
+    </collision>
+    <inertial>
+      <mass value="0.072"/>
+      <inertia ixx="0.00001" ixy="0.0" ixz="0.0" iyy="0.00001" iyz="0.0" izz="0.00001"/>
+    </inertial>
+  </link>
+  <joint name="$(arg prefix)link6_to_camera_mount" type="fixed">
+    <parent link="$(arg prefix)link6"/>
+    <child link="$(arg prefix)camera_mount_link"/>
+    <origin xyz="$(arg cam_x) $(arg cam_y) $(arg cam_z)"
+            rpy="$(arg cam_roll) $(arg cam_pitch) $(arg cam_yaw)"/>
+  </joint>
 </robot>

File: rbpodo_description/robots/rb_6dof.ros2_control.xacro (robot description, xacro)
@@ -4,10 +4,11 @@
     <ros2_control name="RBPodoHardwareInterface" type="system">
       <hardware>
-        <xacro:if value="${use_fake_hardware}">
+        <!-- Xacro may pass Python bool True/False OR string "true"/"false"; handle both -->
+        <xacro:if value="${str(use_fake_hardware).lower() in ('true', '1', 'yes')}">
           <plugin>mock_components/GenericSystem</plugin>
           <param name="mock_sensor_commands">${fake_sensor_commands}</param>
           <param name="state_following_offset">0.0</param>
         </xacro:if>
-        <xacro:unless value="${use_fake_hardware}">
+        <xacro:unless value="${str(use_fake_hardware).lower() in ('true', '1', 'yes')}">
           <plugin>rbpodo_hardware/RBPodoHardwareInterface</plugin>
           <param name="cb_simulation">${cb_simulation}</param>
