Commit message: Revert unnecessary changes.

File: rbpodo_description/robots/rb10_1300e.urdf.xacro (robot description, xacro)
@@ -8,19 +8,9 @@
   <xacro:arg name="use_fake_hardware" default="true"/>
   <xacro:arg name="fake_sensor_commands" default="false"/>
-  <!-- Stereolabs ZED Mini (USB 3, direct-attached) on link6.
-       Default orientation mirrors aw_description/urdf/aw_camera_mount.xacro:
-         zedm +X (lens look) = link6 −Y
-       so the mount uses rpy=(0, 0, −pi/2). -->
-  <!-- Camera mounted on top of TCP, lens facing forward (tcp -Y direction).
-       ZED +X = lens direction → yaw -pi/2 maps cam +X to tcp -Y. -->
   <xacro:arg name="cam_x" default="0.0"/>
   <xacro:arg name="cam_y" default="-0.13"/>
   <xacro:arg name="cam_z" default="0.10"/>
   <xacro:arg name="cam_roll" default="0.0"/>
-  <!-- 25 degrees up -->
-  <!-- <xacro:arg name="cam_pitch" default="0.436332"/>   -->
-  <!-- 22.5 degrees up -->
   <xacro:arg name="cam_pitch" default=".3926996332"/>
-  <!-- <xacro:arg name="cam_yaw" default="-1.5707963267948966"/> -->
   <xacro:arg name="cam_yaw" default="-1.5707963267948966"/>
   <!-- torque_constant = actual_torque_constant * gear_ratio -->
@@ -33,19 +23,4 @@
   <xacro:rb_6dof model_id="rb10_1300e" prefix="$(arg prefix)" tcp_name="tcp" tcp_xyz="0 -0.1153 0" tcp_rpy="0 0 0" />
   <xacro:rb_6dof_ros2_control prefix="$(arg prefix)" robot_ip="$(arg robot_ip)" cb_simulation="$(arg cb_simulation)" use_fake_hardware="$(arg use_fake_hardware)" fake_sensor_commands="$(arg fake_sensor_commands)" torque_constants="${[base_tc, shoulder_tc, elbow_tc, wrist1_tc, wrist2_tc, wrist3_tc]}" />
-  <!-- ══════════════════════════════════════════════════════════════════
-       ZED Mini mount — SELF-CONTAINED.
-       This file used to include `zed_macro.urdf.xacro`, which in turn tried
-       to load `$(find zed_msgs)/meshes/zedm.stl`. On machines where that mesh
-       package/path is missing, RViz reports:
-         "Error retrieving file ... meshes/zedm.stl"
-       and the camera body disappears.
-       To make the robot description robust everywhere, we inline the same
-       ZED frame chain here and render the body as a simple box sized to the
-       real ZED Mini (124.5 x 30.5 x 26.5 mm). The frame names remain identical
-       to Stereolabs' macro so downstream TF/topic consumers still work.
-       Orientation rule for this rig:
-         zedm +X (lens look) = link6 -Y
-       so the mount uses rpy=(0, 0, -pi/2).
-       ══════════════════════════════════════════════════════════════════ -->
   <xacro:property name="M_PI" value="3.1415926535897931"/>
   <link name="$(arg prefix)camera_mount_link">

File: rbpodo_description/robots/rb10_1300e_u.urdf.xacro (robot description, xacro)
@@ -8,12 +8,4 @@
   <xacro:arg name="use_fake_hardware" default="true"/>
   <xacro:arg name="fake_sensor_commands" default="false"/>
-  <!-- Stereolabs ZED Mini on link6 — same mount as rb10_1300e.urdf.xacro.
-       Lens look (zedm +X) = link6 −Y  →  rpy=(0, 0, −π/2) on link6→camera_mount. -->
-  <xacro:arg name="cam_x" default="0.0"/>
-  <xacro:arg name="cam_y" default="-0.08"/>
-  <xacro:arg name="cam_z" default="0.0"/>
-  <xacro:arg name="cam_roll" default="0.0"/>
-  <xacro:arg name="cam_pitch" default="0.0"/>
-  <xacro:arg name="cam_yaw" default="-1.5707963267948966"/>
   <!-- torque_constant = actual_torque_constant * gear_ratio -->
   <xacro:property name="base_tc" value="${1}" />
@@ -23,10 +15,13 @@
   <xacro:property name="wrist2_tc" value="${1}" />
   <xacro:property name="wrist3_tc" value="${1}" />
+  <xacro:arg name="cam_x" default="0.0"/>
+  <xacro:arg name="cam_y" default="-0.08"/>
+  <xacro:arg name="cam_z" default="0.0"/>
+  <xacro:arg name="cam_roll" default="0.0"/>
+  <xacro:arg name="cam_pitch" default="0.0"/>
+  <xacro:arg name="cam_yaw" default="-1.5707963267948966"/>
   <xacro:rb_6dof model_id="rb10_1300e_u" prefix="$(arg prefix)" tcp_name="tcp" tcp_xyz="0 -0.1153 0" tcp_rpy="0 0 0" />
   <xacro:rb_6dof_ros2_control prefix="$(arg prefix)" robot_ip="$(arg robot_ip)" cb_simulation="$(arg cb_simulation)" use_fake_hardware="$(arg use_fake_hardware)" fake_sensor_commands="$(arg fake_sensor_commands)" torque_constants="${[base_tc, shoulder_tc, elbow_tc, wrist1_tc, wrist2_tc, wrist3_tc]}" />
-  <!-- ══════════════════════════════════════════════════════════════════
-       ZED Mini mount — SELF-CONTAINED (no zed_msgs STL). Matches rb10_1300e.
-       ══════════════════════════════════════════════════════════════════ -->
-  <xacro:property name="M_PI" value="3.1415926535897931"/>
+ <xacro:property name="M_PI" value="3.1415926535897931"/>
   <link name="$(arg prefix)camera_mount_link">
     <visual>

File: rbpodo_description/robots/rb_6dof.ros2_control.xacro (robot description, xacro)
@@ -4,11 +4,10 @@
     <ros2_control name="RBPodoHardwareInterface" type="system">
       <hardware>
-        <!-- Xacro may pass Python bool True/False OR string "true"/"false"; handle both -->
-        <xacro:if value="${str(use_fake_hardware).lower() in ('true', '1', 'yes')}">
+        <xacro:if value="${use_fake_hardware}">
           <plugin>mock_components/GenericSystem</plugin>
           <param name="mock_sensor_commands">${fake_sensor_commands}</param>
           <param name="state_following_offset">0.0</param>
         </xacro:if>
-        <xacro:unless value="${str(use_fake_hardware).lower() in ('true', '1', 'yes')}">
+        <xacro:unless value="${use_fake_hardware}">
           <plugin>rbpodo_hardware/RBPodoHardwareInterface</plugin>
           <param name="cb_simulation">${cb_simulation}</param>

File: rbpodo_moveit_config/config/rbpodo.urdf.xacro (robot description, xacro)
@@ -1,13 +1,7 @@
 <?xml version="1.0"?>
-<!--
-  MoveIt no longer uses this file — see launch/moveit.launch.py, which loads
-  $(find rbpodo_description)/robots/<model_id>.urdf.xacro directly.
-  The old wrapper listed several top-level <xacro:arg/> siblings, which is not
-  valid XML (only one document root is allowed) and made xacro fail with
-  "junk after document element" around line 9.
-  This minimal URDF remains so any stale launch or tutorial path still naming
-  config/rbpodo.urdf.xacro gets a parseable file (not a useful robot).
--->
-<robot xmlns:xacro="http://www.ros.org/wiki/xacro" name="rbpodo_moveit_config_unused_stub">
-  <link name="unused_stub_link"/>
+<robot xmlns:xacro="http://www.ros.org/wiki/xacro" name="rb">
+    <xacro:arg name="model_id" default="rb3_730es_u" />
+    <!--robot name="$(arg model_id)"/-->
+    <!-- Import rb urdf file -->
+    <xacro:include filename="$(find rbpodo_description)/robots/$(arg model_id).urdf.xacro" />
 </robot>
