Commit message: Add changes from erdem

File: rbpodo_moveit_config/config/rbpodo.urdf.xacro (robot description, xacro)
@@ -1,7 +1,13 @@
 <?xml version="1.0"?>
-<robot xmlns:xacro="http://www.ros.org/wiki/xacro" name="rb">
-    <xacro:arg name="model_id" default="rb3_730es_u" />
-    <!--robot name="$(arg model_id)"/-->
-    <!-- Import rb urdf file -->
-    <xacro:include filename="$(find rbpodo_description)/robots/$(arg model_id).urdf.xacro" />
+<!--
+  MoveIt no longer uses this file — see launch/moveit.launch.py, which loads
+  $(find rbpodo_description)/robots/<model_id>.urdf.xacro directly.
+  The old wrapper listed several top-level <xacro:arg/> siblings, which is not
+  valid XML (only one document root is allowed) and made xacro fail with
+  "junk after document element" around line 9.
+  This minimal URDF remains so any stale launch or tutorial path still naming
+  config/rbpodo.urdf.xacro gets a parseable file (not a useful robot).
+-->
+<robot xmlns:xacro="http://www.ros.org/wiki/xacro" name="rbpodo_moveit_config_unused_stub">
+  <link name="unused_stub_link"/>
 </robot>
